Commit message: standard MPC tests added.

File: Go2Py/assets/urdf/go2_with_arm.urdf (robot description, URDF)
Before this commit: robot go2, 38 links, 37 joints
Links:
- added link Link6_tip
Joints:
- added joint tip_joint: type fixed, parent Link6, child Link6_tip, origin xyz=0.0 0.0 0.0 rpy=0.0 0.0 0.0

Commit message: Gripper removed and force sensors xmls added.

File: Go2Py/assets/urdf/go2_with_arm.urdf (robot description, URDF)
Before this commit: robot go2, 39 links, 38 joints
Links:
- removed link Link6_tip
- removed link Link7_1
- removed link Link7_2
- added link ef_tip
- link Link6: geometry visual mesh filename=d1_assets/stl/Link6-new.stl
Joints:
- removed joint Joint7_1
- removed joint Joint7_2
- joint tip_joint: child Link6_tip -> ef_tip; origin xyz=0.0 0.0 0.0 rpy=0.0 0.0 0.0 -> xyz=0.0 0.0 0.053 rpy=0.0 0.0 0.0
