Commit message: visualization assets added

File: Go2Py/assets/urdf/d1_description.urdf (robot description, URDF)
Before this commit: robot d1_description, 9 links, 8 joints
Links:
- removed link Link7_1
- removed link Link7_2
- link Link1: geometry collision mesh filename=d1_assets/stl/Link1.STL; visual mesh filename=d1_assets/stl/Link1.STL
- link Link2: geometry collision mesh filename=d1_assets/stl/Link2.STL; visual mesh filename=d1_assets/stl/Link2.STL
- link Link3: geometry collision mesh filename=d1_assets/stl/Link3.STL; visual mesh filename=d1_assets/stl/Link3.STL
- link Link4: geometry collision mesh filename=d1_assets/stl/Link4.STL; visual mesh filename=d1_assets/stl/Link4.STL
- link Link5: geometry collision mesh filename=d1_assets/stl/Link5.STL; visual mesh filename=d1_assets/stl/Link5.STL
- link Link6: geometry visual mesh filename=d1_assets/stl/Link6-new.stl
- link base_link: geometry collision mesh filename=d1_assets/stl/base_link.STL; visual mesh filename=d1_assets/stl/base_link.STL
Joints:
- removed joint Joint7_1
- removed joint Joint7_2
